Commit message: Rename WidowX mesh files, OBJ groups and materials to valid USD identifiers
Isaac Sim's URDF importer names prims after mesh files, OBJ object groups
and material names. The vendored meshes were named WXSA-250-M-1-Base with
hyphens and the materials Material.018 with dots, neither of which is a
valid prim name, and the importer failed with 'Used null prim'. Use
underscores throughout and update the URDF references.

Co-Authored-By: Claude Fable 5.1 <noreply@anthropic.com>
Claude-Session: https://claude.ai/code/session_0142xgjULv5btKafEG5sU6WB

File: gen3_isaac_env/gen3/assets/widowx/wx250s.urdf (robot description, URDF)
Before this commit: robot wx250s, 14 links, 13 joints
Links:
- link base_link: geometry collision mesh filename=meshes_wx250s/WXSA_250_M_1_Base.stl scale=0.001 0.001 0.001; visual mesh filename=meshes_wx250s/WXSA_250_M_1_Base.obj scale=0.001 0.001 0.001
- link gripper_bar_link: geometry collision mesh filename=meshes_wx250s/WXSA_250_M_9_Gripper_Bar.stl scale=0.001 0.001 0.001; visual mesh filename=meshes_wx250s/WXSA_250_M_9_Gripper_Bar.obj scale=0.001 0.001 0.001
- link gripper_link: geometry collision mesh filename=meshes_wx250s/WXSA_250_M_7_Gripper.stl scale=0.001 0.001 0.001; visual mesh filename=meshes_wx250s/WXSA_250_M_7_Gripper.obj scale=0.001 0.001 0.001
- link gripper_prop_link: geometry collision mesh filename=meshes_wx250s/WXSA_250_M_8_Gripper_Prop.stl scale=0.001 0.001 0.001; visual mesh filename=meshes_wx250s/WXSA_250_M_8_Gripper_Prop.obj scale=0.001 0.001 0.001
- link left_finger_link: geometry collision mesh filename=meshes_wx250s/WXSA_250_M_10_Finger.stl scale=0.001 0.001 0.001; visual mesh filename=meshes_wx250s/WXSA_250_M_10_Finger.obj scale=0.001 0.001 0.001
- link lower_forearm_link: geometry collision mesh filename=meshes_wx250s/WXSA_250_M_5_LF.stl scale=0.001 0.001 0.001; visual mesh filename=meshes_wx250s/WXSA_250_M_5_LF.obj scale=0.001 0.001 0.001
- link right_finger_link: geometry collision mesh filename=meshes_wx250s/WXSA_250_M_10_Finger.stl scale=0.001 0.001 0.001; visual mesh filename=meshes_wx250s/WXSA_250_M_10_Finger.obj scale=0.001 0.001 0.001
- link shoulder_link: geometry collision mesh filename=meshes_wx250s/WXSA_250_M_2_Shoulder.stl scale=0.001 0.001 0.001; visual mesh filename=meshes_wx250s/WXSA_250_M_2_Shoulder.obj scale=0.001 0.001 0.001
- link upper_arm_link: geometry collision mesh filename=meshes_wx250s/WXSA_250_M_3_UA.stl scale=0.001 0.001 0.001; visual mesh filename=meshes_wx250s/WXSA_250_M_3_UA.obj scale=0.001 0.001 0.001
- link upper_forearm_link: geometry collision mesh filename=meshes_wx250s/WXSA_250_M_4_UF.stl scale=0.001 0.001 0.001; visual mesh filename=meshes_wx250s/WXSA_250_M_4_UF.obj scale=0.001 0.001 0.001
- link wrist_link: geometry collision mesh filename=meshes_wx250s/WXSA_250_M_6_Wrist.stl scale=0.001 0.001 0.001; visual mesh filename=meshes_wx250s/WXSA_250_M_6_Wrist.obj scale=0.001 0.001 0.001
